Commit message: Nav2 fonctionnel avec rviz

File: src/car/model/gazebo.xacro (robot description, xacro)
@@ -15,5 +15,5 @@
         <sensor name="lidar" type="gpu_lidar">
             <pose relative_to="lidar_link">0 0 0 0 0 0</pose>
-            <topic>scan</topic>
+            <topic>/scan</topic>
             <update_rate>10</update_rate>
             <gz_frame_id>lidar_link</gz_frame_id>

File: src/car/model/robot.xacro (robot description, xacro)
@@ -71,5 +71,5 @@
                 <visual>
                         <geometry>
-                                <box size="0.5 0.1 0.5"/>
+                                <box size="0.1 0.1 0.1"/>
                         </geometry>
                         <origin xyz="0 0 0" rpy="0 0 0"/>
@@ -98,5 +98,5 @@
                 <visual>
                         <geometry>
-                                <box size="0.5 0.1 0.5"/>
+                                <box size="0.1 0.1 0.1"/>
                         </geometry>
                         <origin xyz="0 0 0" rpy="0 0 0"/>
@@ -125,5 +125,5 @@
                 <visual>
                         <geometry>
-                                <box size="0.5 0.1 0.5"/>
+                                <box size="0.1 0.1 0.1"/>
                         </geometry>
                         <origin xyz="0 0 0" rpy="0 0 0"/>
@@ -152,5 +152,5 @@
                 <visual>
                         <geometry>
-                                <box size="0.5 0.1 0.5"/>
+                                <box size="0.1 0.1 0.1"/>
                         </geometry>
                         <origin xyz="0 0 0" rpy="0 0 0"/>
@@ -160,5 +160,5 @@
                 <parent link="base_link"/>
                 <child link="rb_link"/>
-                <origin xyz="-0.5 0.5 -0.25" rpy="0 0 0"/>
+                <origin xyz="-0.5 -0.5 -0.25" rpy="0 0 0"/>
                 <axis xyz="0 1 0"/>
                 <dynamics damping="1.0" friction="1.0"/>
@@ -168,10 +168,10 @@
                 <parent link="rb_link"/>
                 <child link="rb_rotation_link"/>
-                <origin xyz="0 0 0" rpy="0 0 0"/>
+                <origin xyz="0 0.1 0" rpy="0 0 0"/>
         </joint>
         <joint name="rf_joint" type="continuous">
                 <parent link="base_link"/>
                 <child link="rf_link"/>
-                <origin xyz="0.5 0.5 -0.25" rpy="0 0 0"/>
+                <origin xyz="0.5 -0.5 -0.25" rpy="0 0 0"/>
                 <axis xyz="0 1 0"/>
                 <dynamics damping="1.0" friction="1.0"/>
@@ -181,10 +181,10 @@
                 <parent link="rf_link"/>
                 <child link="rf_rotation_link"/>
-                <origin xyz="0 0 0" rpy="0 0 0"/>
+                <origin xyz="0 0.1 0" rpy="0 0 0"/>
         </joint>
         <joint name="lb_joint" type="continuous">
                 <parent link="base_link"/>
                 <child link="lb_link"/>
-                <origin xyz="-0.5 -0.5 -0.25" rpy="0 0 0"/>
+                <origin xyz="-0.5 0.5 -0.25" rpy="0 0 0"/>
                 <axis xyz="0 1 0"/>
                 <dynamics damping="1.0" friction="1.0"/>
@@ -194,10 +194,10 @@
                 <parent link="lb_link"/>
                 <child link="lb_rotation_link"/>
-                <origin xyz="0 0 0" rpy="0 0 0"/>
+                <origin xyz="0 -0.1 0" rpy="0 0 0"/>
         </joint>
         <joint name="lf_joint" type="continuous">
                 <parent link="base_link"/>
                 <child link="lf_link"/>
-                <origin xyz="0.5 -0.5 -0.25" rpy="0 0 0"/>
+                <origin xyz="0.5 0.5 -0.25" rpy="0 0 0"/>
                 <axis xyz="0 1 0"/>
                 <dynamics damping="1.0" friction="1.0"/>
@@ -207,5 +207,5 @@
                 <parent link="lf_link"/>
                 <child link="lf_rotation_link"/>
-                <origin xyz="0 0 0" rpy="0 0 0"/>
+                <origin xyz="0 -0.1 0" rpy="0 0 0"/>
         </joint>
         <!-- LIDAR -->

Commit message: Passage en roues holonomes

File: src/car/model/gazebo.xacro (robot description, xacro)
@@ -45,5 +45,5 @@
         <mu1>1.5</mu1>
         <mu2>0.5</mu2>  <!-- MU2 TRÈS FAIBLE -->
-        <fdir1>0 1 0</fdir1>  <!-- Direction de friction primaire = axe de rotation -->
+        <fdir1>0 -1 0</fdir1>  <!-- Direction de friction primaire = axe de rotation -->
         <kp>10000000.0</kp>
         <kd>10.0</kd>
@@ -55,5 +55,5 @@
         <mu1>1.5</mu1>
         <mu2>0.5</mu2>
-        <fdir1>0 1 0</fdir1>
+        <fdir1>0 -1 0</fdir1>
         <kp>10000000.0</kp>
         <kd>10.0</kd>

File: src/car/model/robot.xacro (robot description, xacro)
@@ -160,6 +160,6 @@
                 <parent link="base_link"/>
                 <child link="rb_link"/>
-                <origin xyz="-0.5 -0.5 -0.25" rpy="0 0 0"/>
-                <axis xyz="0 1 0"/>
+                <origin xyz="-0.5 -0.5 -0.25" rpy="0 0 ${-pi/4}"/>
+                <axis xyz="0 -1 0"/>
                 <dynamics damping="1.0" friction="1.0"/>
                 <limit effort="1000" velocity="1000"/>
@@ -168,11 +168,11 @@
                 <parent link="rb_link"/>
                 <child link="rb_rotation_link"/>
-                <origin xyz="0 0.1 0" rpy="0 0 0"/>
+                <origin xyz="0 -0.1 0" rpy="0 0 0"/>
         </joint>
         <joint name="rf_joint" type="continuous">
                 <parent link="base_link"/>
                 <child link="rf_link"/>
-                <origin xyz="0.5 -0.5 -0.25" rpy="0 0 0"/>
-                <axis xyz="0 1 0"/>
+                <origin xyz="0.5 -0.5 -0.25" rpy="0 0 ${pi/4}"/>
+                <axis xyz="0 -1 0"/>
                 <dynamics damping="1.0" friction="1.0"/>
                 <limit effort="1000" velocity="1000"/>
@@ -181,10 +181,10 @@
                 <parent link="rf_link"/>
                 <child link="rf_rotation_link"/>
-                <origin xyz="0 0.1 0" rpy="0 0 0"/>
+                <origin xyz="0 -0.1 0" rpy="0 0 0"/>
         </joint>
         <joint name="lb_joint" type="continuous">
                 <parent link="base_link"/>
                 <child link="lb_link"/>
-                <origin xyz="-0.5 0.5 -0.25" rpy="0 0 0"/>
+                <origin xyz="-0.5 0.5 -0.25" rpy="0 0 ${pi/4}"/>
                 <axis xyz="0 1 0"/>
                 <dynamics damping="1.0" friction="1.0"/>
@@ -194,10 +194,10 @@
                 <parent link="lb_link"/>
                 <child link="lb_rotation_link"/>
-                <origin xyz="0 -0.1 0" rpy="0 0 0"/>
+                <origin xyz="0 0.1 0" rpy="0 0 0"/>
         </joint>
         <joint name="lf_joint" type="continuous">
                 <parent link="base_link"/>
                 <child link="lf_link"/>
-                <origin xyz="0.5 0.5 -0.25" rpy="0 0 0"/>
+                <origin xyz="0.5 0.5 -0.25" rpy="0 0 ${-pi/4}"/>
                 <axis xyz="0 1 0"/>
                 <dynamics damping="1.0" friction="1.0"/>
@@ -207,5 +207,5 @@
                 <parent link="lf_link"/>
                 <child link="lf_rotation_link"/>
-                <origin xyz="0 -0.1 0" rpy="0 0 0"/>
+                <origin xyz="0 0.1 0" rpy="0 0 0"/>
         </joint>
         <!-- LIDAR -->
