Commit message: maj trajectoires

File: src/car/model/real-robot/robot.xacro (robot description, xacro)
@@ -45,5 +45,5 @@
                 <parent link="base_footprint"/>
                 <child link="base_link"/>
-                <origin xyz="0 0 0.5" rpy="0 0 0"/>
+                <origin xyz="0 0 0.5" rpy="0 0 ${pi}"/>
         </joint>
         <link name="front_visual">
@@ -57,5 +57,5 @@
                 <parent link="base_link"/>
                 <child link="front_visual"/>
-                <origin xyz="0.5 0 0.15" rpy="0 0 0"/>
+                <origin xyz="-0.5 0 0.15" rpy="0 0 0"/>
         </joint>
         <!-- WHEELS -->
@@ -171,6 +171,6 @@
                 <parent link="base_link"/>
                 <child link="rb_link"/>
-                <origin xyz="-0.5 -0.5 -0.25" rpy="0 0 ${-pi/4}"/>
-                <axis xyz="0 -1 0"/>
+                <origin xyz="0.5 0.5 -0.25" rpy="0 0 ${-pi/4}"/>
+                <axis xyz="0 1 0"/>
                 <dynamics damping="1.0" friction="1.0"/>
                 <limit effort="1000" velocity="1000"/>
@@ -184,6 +184,6 @@
                 <parent link="base_link"/>
                 <child link="rf_link"/>
-                <origin xyz="0.5 -0.5 -0.25" rpy="0 0 ${pi/4}"/>
-                <axis xyz="0 -1 0"/>
+                <origin xyz="-0.5 0.5 -0.25" rpy="0 0 ${pi/4}"/>
+                <axis xyz="0 1 0"/>
                 <dynamics damping="1.0" friction="1.0"/>
                 <limit effort="1000" velocity="1000"/>
@@ -197,5 +197,5 @@
                 <parent link="base_link"/>
                 <child link="lb_link"/>
-                <origin xyz="-0.5 0.5 -0.25" rpy="0 0 ${pi/4}"/>
+                <origin xyz="0.5 -0.5 -0.25" rpy="0 0 ${pi/4}"/>
                 <axis xyz="0 1 0"/>
                 <dynamics damping="1.0" friction="1.0"/>
@@ -210,5 +210,5 @@
                 <parent link="base_link"/>
                 <child link="lf_link"/>
-                <origin xyz="0.5 0.5 -0.25" rpy="0 0 ${-pi/4}"/>
+                <origin xyz="-0.5 -0.5 -0.25" rpy="0 0 ${-pi/4}"/>
                 <axis xyz="0 1 0"/>
                 <dynamics damping="1.0" friction="1.0"/>
